File: project/project.kicad_sch (KiCad schematic)
At the start: 0 parts

Commit message: hierarchical sheets
Other:
- added sheet DDR3L (ddr3l.kicad_sch)
- added sheet Display (display.kicad_sch)
- added sheet IO expander (io-expander.kicad_sch)
- added sheet MPU (mpu.kicad_sch)
- added sheet Power & Decoupling (power-decoupling.kicad_sch)
- added sheet USB C DRP (usb-c-drp.kicad_sch)
- added sheet WLAN & Bluetooth (ESP32) (wlan-and-ble.kicad_sch)
