File: project/power-decoupling.kicad_sch (KiCad schematic)
At the start: 0 parts

Commit message: Added CubeMX project and some schematic components are added
Parts:
- added C16, C18, C20, C22, C26: 10u, bozi:GRT18_T15, symbol Device:C
- added C17, C19, C21, C23, C27, C28, C67, C68, C76, C77: 22u, bozi:GRM18_T20, symbol Device:C
- added C24, C25, C30, C32: 1u, bozi:GRM15_T05, symbol Device:C
- added C29, C31, C33, C34, C35, C36: 4u7, bozi:GRM15_T15, symbol Device:C
- added C37, C38, C39, C40, C41, C42, C43, C44, C45, C46, C47, C56, C57, C58, C59, C60, C61, C62, C63, C64, C65, C66, C69, C70, C71, C72, C73, C74, C75: 1u, bozi:GRM03_T09, symbol Device:C
- added C48: 10n, bozi:GRM15_T05, symbol Device:C
- added C49, C50, C51, C52, C53, C54, C55: 1n, bozi:GRM03_T03, symbol Device:C
- added IC2: LM66200DRLR, SOTFL50P160X60-8N, symbol bozi:LM66200DRLR
- added IC3: STPMIC1DPQR, bozi:QFN40P500X600X80-45N-D_edit, symbol bozi:STPMIC1DPQR
- added IC4: ST1S31PUR, bozi:SON65P300X300X100-9N-D_edit, symbol bozi:ST1S31PUR
- added L1, L2, L3, L4: 1µ, bozi:DFE2HCAH1R0MJ0L_edit, symbol Device:L
- added L5: 2u2, bozi:INDPM4040X250N_edit, symbol Device:L
- added R4: 560, bozi:RESC1005X37N_edit, symbol Device:R
- added R5: 75k, bozi:RESC1005X37N_edit, symbol Device:R
- added R6: 24k, bozi:RESC1005X37N_edit, symbol Device:R
- added R7: 100m, bozi:RESC2012X60N_edit, symbol Device:R
- added SW1: SW_Push, bozi:PTS636SM43SMTRLFS_edit, symbol Switch:SW_Push
- added TP1, TP10, TP2, TP3, TP4, TP5, TP6, TP7, TP8, TP9: TestPoint, TestPoint:TestPoint_Pad_D1.0mm, symbol Connector:TestPoint
Connections:
- new net: IC3.7 (VLX1), L1.2
- new net: IC4.5 (PG), R4.1
- new net: IC4.3 (FB), R5.1, R6.2
- new net: IC4.7 (SW), L5.1
- new net: C36.1, IC3.39 (LDO4OUT), R7.1, TP10.1
- new net: C35.2, IC3.40 (INTLDO)
- new net: C48.1, IC3.17 (PONKEYN), SW1.1
- new net: IC3.25 (VLX4), L4.1
- new net: C31.1, IC3.18 (LDO2OUT), TP8.1
- new net: IC3.11 (VLX2), L2.2
- new net: IC3.29 (VLX3), L3.1
- new net 3V3_AO: C27.1, C28.1, IC3.37 (SWIN), L5.2, R4.2, R5.2, TP5.1
- new net 3V3_SW: IC3.38 (SWOUT)
- new net 5V_VIN: C16.1, C18.1, C20.1, C22.1, C25.1, C26.1, C30.1, C32.1, C34.2, IC3.12 (BUCK2IN), IC3.19 (LDO25IN), IC3.22 (LDO16IN), IC3.24 (BUCK4IN), IC3.28 (BUCK3IN), IC3.36 (VIN), IC3.8 (BUCK1IN), IC4.1 (VINA), IC4.6 (VINSW)
- new net GNDREF: C16.2, C17.2, C18.2, C19.2, C20.2, C21.2, C22.2, C23.2, C24.2, C25.2, C26.2, C27.2, C28.2, C29.2, C30.2, C31.2, C32.2, C33.2, C34.1, C35.1, C36.2, C37.2, C38.2, C39.2, C40.2, C41.2, C42.2, C43.2, C44.2, C45.2, C46.2, C47.2, C48.2, C49.2, C50.2, C51.2, C52.2, C53.2, C54.2, C55.2, C56.2, C57.2, C58.2, C59.2, C60.2, C61.2, C62.2, C63.2, C64.2, C65.2, C66.2, C67.2, C68.2, C69.2, C70.2, C71.2, C72.2, C73.2, C74.2, C75.2, C76.2, C77.2, IC2.1 (GND_1), IC2.5 (GND_2), IC3.10 (PGND2), IC3.13 (LDO3IN), IC3.15 (GNDLDO), IC3.26 (PGND4), IC3.30 (PGND3), IC3.32 (PGBOOST), IC3.41 (AGND), IC3.45 (EPGND), IC3.6 (PGND1), IC4.4 (AGND), IC4.8 (PGND), IC4.9 (EP), R6.1, SW1.2
- new net I2C_SCL: IC3.4 (SCL)
- new net I2C_SDA: IC3.3 (SDA)
- new net INT_N: IC3.43 (~{INT})
- new net NRST: IC3.1 (~{RST})
- new net PMIC_WAKEUP: IC3.2 (WAKEUP)
- new net PWR_ON: IC3.44 (PWRCTRL)
- new net VBAT: IC2.6 (VIN2)
- new net VBUS: IC2.3 (VIN1)
- new net VDD: C21.1, C37.1, C38.1, C39.1, C40.1, C41.1, C42.1, C43.1, C44.1, C45.1, C46.1, C47.1, IC3.31 (VOUT3), IC3.42 (VIO), IC4.2 (EN), L3.2, TP3.1
- new net VDD_ADC: C29.1, IC3.23 (LDO1OUT), TP7.1
- new net VDD_CORE: C23.1, C59.1, C60.1, C61.1, C62.1, C63.1, C64.1, C65.1, C66.1, C67.1, C68.1, IC3.27 (VOUT4), L4.2, TP4.1
- new net VDD_CPU: C17.1, C69.1, C70.1, C71.1, C72.1, C73.1, C74.1, C75.1, C76.1, C77.1, IC3.5 (VOUT1), L1.1, TP1.1
- new net VDD_DDR: C19.1, C49.1, C50.1, C51.1, C52.1, C53.1, C54.1, C55.1, C56.1, C57.1, C58.1, IC3.9 (VOUT2), L2.1, TP2.1
- new net VDD_SD: C33.1, IC3.20 (LDO5OUT), TP9.1
- new net VDD_USB: R7.2
- new net VREF_DDR: C24.1, IC3.16 (VREFDDR), TP6.1
- new net VSYS: IC2.2 (VOUT_1), IC2.7 (VOUT_2)
- no-connect marks 0 -> 5
Other:
- note added: "3V3 Always on"
- note added: "Decoupling capacitors (CPU)"
- note added: "MAX 2.5 A forward voltage"

Commit message: schemtic is done, need to go through BOM
Parts:
- removed IC2: LM66200DRLR, SOTFL50P160X60-8N, symbol bozi:LM66200DRLR
- C19: renamed from C16; value 10u -> 10uF; Manufacturer_Name (none) -> Murata Electronics
- C20: renamed from C17; value 22u -> 22uF; Manufacturer_Name (none) -> Murata Electronics
- C21: renamed from C18; value 10u -> 10uF; Manufacturer_Name (none) -> Murata Electronics
- C22: renamed from C19; value 22u -> 22uF; Manufacturer_Name (none) -> Murata Electronics
- C23: renamed from C20; value 10u -> 10uF; Manufacturer_Name (none) -> Murata Electronics
- C24: renamed from C21; value 22u -> 22uF; Manufacturer_Name (none) -> Murata Electronics
- C25: renamed from C22; value 10u -> 10uF; Manufacturer_Name (none) -> Murata Electronics
- C26: renamed from C23; value 22u -> 22uF; Manufacturer_Name (none) -> Murata Electronics
- C27: renamed from C24; value 1u -> 1uF; Manufacturer_Name (none) -> Murata Electronics
- C28: renamed from C25; value 1u -> 1uF; Manufacturer_Name (none) -> Murata Electronics
- C29: renamed from C26; value 10u -> 10uF; Manufacturer_Name (none) -> Murata Electronics
- C30: renamed from C27; value 22u -> 22uF; Manufacturer_Name (none) -> Murata Electronics
- C31: renamed from C28; value 22u -> 22uF; Manufacturer_Name (none) -> Murata Electronics
- C32: renamed from C29; value 4u7 -> 4.7uF; Manufacturer_Name (none) -> Murata Electronics
- C33: renamed from C30; value 1u -> 1uF; Manufacturer_Name (none) -> Murata Electronics
- C34: renamed from C31; value 4u7 -> 4.7uF; Manufacturer_Name (none) -> Murata Electronics
- C35: renamed from C32; value 1u -> 1uF; Manufacturer_Name (none) -> Murata Electronics
- C36: renamed from C33; value 4u7 -> 4.7uF; Manufacturer_Name (none) -> Murata Electronics
- C37: renamed from C34; value 4u7 -> 4.7uF; Manufacturer_Name (none) -> Murata Electronics
- C38: renamed from C35; value 4u7 -> 4.7uF; Manufacturer_Name (none) -> Murata Electronics
- C39: renamed from C36; value 4u7 -> 4.7uF; Manufacturer_Name (none) -> Murata Electronics
- C40: renamed from C37; value 1u -> 1uF; Manufacturer_Name (none) -> Murata Electronics
- C41: renamed from C38; value 1u -> 1uF; Manufacturer_Name (none) -> Murata Electronics
- C42: renamed from C39; value 1u -> 1uF; Manufacturer_Name (none) -> Murata Electronics
- C43: renamed from C40; value 1u -> 1uF; Manufacturer_Name (none) -> Murata Electronics
- C44: renamed from C41; value 1u -> 1uF; Manufacturer_Name (none) -> Murata Electronics
- C45: renamed from C42; value 1u -> 1uF; Manufacturer_Name (none) -> Murata Electronics
- C46: renamed from C43; value 1u -> 1uF; Manufacturer_Name (none) -> Murata Electronics
- C47: renamed from C44; value 1u -> 1uF; Manufacturer_Name (none) -> Murata Electronics
- C48: renamed from C45; value 1u -> 1uF; Manufacturer_Name (none) -> Murata Electronics
- C49: renamed from C46; value 1u -> 1uF; Manufacturer_Name (none) -> Murata Electronics
- C51: renamed from C48; value 10n -> 100nF; footprint bozi:GRM15_T05 -> bozi:GRM18_T10; Manufacturer_Name (none) -> Murata Electronics; Manufacturer_Part_Number GRM155R71H103KA88D -> GRM188R71H104KA93D
- C52: renamed from C49; value 1n -> 1nF; Manufacturer_Name (none) -> Murata Electronics
- C53: renamed from C50; value 1n -> 1nF; Manufacturer_Name (none) -> Murata Electronics
- C54: renamed from C51; value 1n -> 1nF; Manufacturer_Name (none) -> Murata Electronics
- C55: renamed from C52; value 1n -> 1nF; Manufacturer_Name (none) -> Murata Electronics
- C56: renamed from C53; value 1n -> 1nF; Manufacturer_Name (none) -> Murata Electronics
- C57: renamed from C54; value 1n -> 1nF; Manufacturer_Name (none) -> Murata Electronics
- C58: renamed from C55; value 1n -> 1nF; Manufacturer_Name (none) -> Murata Electronics
- C59: renamed from C56; value 1u -> 1uF; Manufacturer_Name (none) -> Murata Electronics
- C60: renamed from C57; value 1u -> 1uF; Manufacturer_Name (none) -> Murata Electronics
- C61: renamed from C58; value 1u -> 1uF; Manufacturer_Name (none) -> Murata Electronics
- C62: renamed from C59; value 1u -> 1uF; Manufacturer_Name (none) -> Murata Electronics
- C63: renamed from C60; value 1u -> 1uF; Manufacturer_Name (none) -> Murata Electronics
- C64: renamed from C61; value 1u -> 1uF; Manufacturer_Name (none) -> Murata Electronics
- C65: renamed from C62; value 1u -> 1uF; Manufacturer_Name (none) -> Murata Electronics
- C66: renamed from C63; value 1u -> 1uF; Manufacturer_Name (none) -> Murata Electronics
- C67: renamed from C64; value 1u -> 1uF; Manufacturer_Name (none) -> Murata Electronics
- C68: renamed from C65; value 1u -> 1uF; Manufacturer_Name (none) -> Murata Electronics
- C69: renamed from C66; value 1u -> 1uF; Manufacturer_Name (none) -> Murata Electronics
- C70: renamed from C67; value 22u -> 22uF; Manufacturer_Name (none) -> Murata Electronics
- C72: renamed from C69; value 1u -> 1uF; Manufacturer_Name (none) -> Murata Electronics
- C73: renamed from C70; value 1u -> 1uF; Manufacturer_Name (none) -> Murata Electronics
- C74: renamed from C71; value 1u -> 1uF; Manufacturer_Name (none) -> Murata Electronics
- C75: renamed from C72; value 1u -> 1uF; Manufacturer_Name (none) -> Murata Electronics
- C76: renamed from C73; value 1u -> 1uF; Manufacturer_Name (none) -> Murata Electronics
- C77: renamed from C74; value 1u -> 1uF; Manufacturer_Name (none) -> Murata Electronics
- C78: renamed from C75; value 1u -> 1uF; Manufacturer_Name (none) -> Murata Electronics
- C79: renamed from C76; value 22u -> 22uF; Manufacturer_Name (none) -> Murata Electronics
- C80: renamed from C77; value 22u -> 22uF; Manufacturer_Name (none) -> Murata Electronics
- L1, L2, L3, L4: value 1µ -> 1uH; Manufacturer_Name (none) -> Murata Electronics; Manufacturer_Part_Number DFE252012P-1ROM=P2 -> DFE252012P-1R0M=P2
- L5: value 2u2 -> 2.2uH; Manufacturer_Name (none) -> Würth Elektronik
- R10: renamed from R6; Manufacturer_Name (none) -> YAGEO
- R11: renamed from R7; Manufacturer_Name (none) -> Yageo
- R8: renamed from R4; value 560 -> 560R; Manufacturer_Name (none) -> YAGEO
- R9: renamed from R5; Manufacturer_Name (none) -> YAGEO
- SW1: value SW_Push -> PTS636SM43SMTR LFS; Manufacturer_Name (none) -> C&K; Manufacturer_Part_Number FSM6JSMATR_SW_5-1437565-0 -> PTS636SM43SMTR LFS
- renumbered C47 to C50, C68 to C71, TP5 to TP10, TP6 to TP11, TP7 to TP12, TP8 to TP13, TP9 to TP14, TP10 to TP15, TP1 to TP6, TP2 to TP7, TP3 to TP8, TP4 to TP9
Connections:
- net INT_N renamed PMIC_INT_N
Other:
- note removed: "MAX 2.5 A forward voltage"

Commit message: schemtic is done, annotation set
Parts:
- removed C28: 1uF, bozi:GRM15_T05, symbol Device:C
- removed C29: 10uF, bozi:GRT18_T15, symbol Device:C
- removed C30, C31: 22uF, bozi:GRM18_T20, symbol Device:C
- removed IC4: ST1S31PUR, bozi:SON65P300X300X100-9N-D_edit, symbol bozi:ST1S31PUR
- removed L5: 2.2uH, bozi:INDPM4040X250N_edit, symbol Device:L
- removed R10: 24k, bozi:RESC1005X37N_edit, symbol Device:R
- removed R8: 560R, bozi:RESC1005X37N_edit, symbol Device:R
- removed R9: 75k, bozi:RESC1005X37N_edit, symbol Device:R
- added BT1: Battery_Cell, symbol Device:Battery_Cell
- added C70: 4.7uF, bozi:GRM15_T15, symbol Device:C
- added C78, C79: 4.7uF, bozi:GRM18_T15, symbol Device:C
- added C80, C81: 10uF, bozi:GRT18_T15, symbol Device:C
- added C82: 470pF, bozi:GRT15_T05, symbol Device:C
- added D2: LED, bozi:LEDC1608X70N_edit, symbol Device:LED
- added IC3: MAX17262REWL+T, BGA9C40P3X3_147X145X69, symbol bozi:MAX17262REWL+T
- added IC4: LD39200PU33R, SON95P300X300X100-7N-D, symbol bozi:LD39200PU33R
- added IC5: TPS2117DRLR, SOTFL50P160X60-8N, symbol bozi:TPS2117DRLR
- added R11, R12, R13, R14, R18, R19, R20, R21, R22: 0R, bozi:RESC1005X37N_edit, symbol Device:R
- added R15, R17: 1k, bozi:RESC1005X37N_edit, symbol Device:R
- added R16: 240R, bozi:RESC1005X37N_edit, symbol Device:R
- added TH1: 10k NTC, bozi:THRMC1005X55N, symbol Device:Thermistor_NTC
- added TP8: TestPoint, TestPoint:TestPoint_Pad_D1.0mm, symbol Connector:TestPoint
- added U2: MCP73831-2-OT, Package_TO_SOT_SMD:SOT-23-5, symbol bozi:MCP73831-2-OT
- renumbered C40 to C20, C41 to C21, C42 to C22, C43 to C23, C44 to C24, C45 to C25, C46 to C26, C47 to C27, C48 to C28, C49 to C29, C50 to C30, C20 to C31, C21 to C32, C22 to C33, C52 to C34, C53 to C35, C54 to C36, C55 to C37, C56 to C38, C57 to C39, C58 to C40, C59 to C41, C60 to C42, C61 to C43, C23 to C44, C24 to C45, C25 to C46, C26 to C47, C62 to C48, C63 to C49, C64 to C50, C65 to C51, C66 to C52, C67 to C53, C68 to C54, C69 to C55, C70 to C56, C71 to C57, C72 to C58, C73 to C59, C74 to C60, C75 to C61, C76 to C62, C77 to C63, C78 to C64, C79 to C65, C80 to C66, C27 to C67, C32 to C68, C33 to C69, C34 to C71, C35 to C72, C36 to C73, C37 to C74, C38 to C75, C39 to C76, C51 to C77, IC3 to IC2, R11 to R10, TP14 to TP10, TP15 to TP11, TP10 to TP12, TP6 to TP2, TP7 to TP3, TP8 to TP4, TP9 to TP5, TP11 to TP6, TP12 to TP7, TP13 to TP9
Connections:
- net 3V3_AO: now also C80.1, IC4.1 (OUT), IC4.2 (ADJ/SENSE); no longer IC2.37 (SWIN)
- net 5V_VIN: now also R12.1, R19.1, R20.1; no longer C19.1, C32.1, C44.1, C46.1, C69.1, C72.1, C74.2, IC2.12 (BUCK2IN), IC2.19 (LDO25IN), IC2.22 (LDO16IN), IC2.24 (BUCK4IN), IC2.28 (BUCK3IN), IC2.36 (VIN), IC2.8 (BUCK1IN)
- net GNDREF: now also C70.2, C80.2, C81.2, IC4.3 (GND), IC4.7 (EPAD), IC5.1 (GND), IC5.4 (PR1), IC5.5 (MODE)
- net VDD_CODEC: now reaches IC2.21 (LDO6OUT)
- net VDD_CODEC: now also C70.1, TP8.1
- net 3V3_SW: no longer names the net of IC2.38 (SWOUT)
- new net: IC3.B3 (SYS), R14.1
- new net: R15.2, R17.1
- new net: C82.1, IC3.C2 (REG)
- new net: IC5.3 (VIN1), R22.2
- new net: BT1.1 (+), C79.1, R11.1, R13.1, U2.3 (V_{BAT})
- new net: IC5.2 (VOUT_1), IC5.7 (VOUT_2), R21.2
- new net: IC5.6 (VIN2), R20.2
- new net: D2.1 (K), R16.1
- new net: R16.2, U2.1 (STAT)
- new net: IC3.A2 (BATT), R13.2
- new net: C78.1, D2.2 (A), R12.2, U2.4 (V_{DD})
- new net: IC3.A1 (TH), TH1.1
- new net: R15.1, U2.5 (PROG)
- new net 3V3_PG: IC4.4 (PG)
- new net BFG_ALRT: IC3.B2 (ALRT)
- new net BFG_SCL: IC3.B1 (SCL)
- new net BFG_SDA: IC3.C1 (SDA)
- new net GND: BT1.2 (-), C78.2, C79.2, C82.2, IC3.C3 (GND), R17.2, TH1.2, U2.2 (V_{SS})
- new net VBAT: R11.2, R14.2, R18.1, R22.1
- new net VSOURCE_IO: IC5.8 (ST)
- new net VSYS: C19.1, C32.1, C44.1, C46.1, C69.1, C72.1, C74.2, C81.1, IC2.12 (BUCK2IN), IC2.19 (LDO25IN), IC2.22 (LDO16IN), IC2.24 (BUCK4IN), IC2.28 (BUCK3IN), IC2.36 (VIN), IC2.8 (BUCK1IN), IC4.5 (EN), IC4.6 (IN), R18.2, R19.2, R21.1
- no-connect marks 5 -> 7
Other:
- note added: "Battery charger"
- note added: "Battery charger and battery fuel gauge"
- note added: "Battery fuel gauge"
- note added: "Pads for VBAT and GND"
- note added: "Power source MUX"
- moved on the sheet: C20, C21, C22, C23, C24, C25, C26, C27, C28, C29, C30, C34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
